File: output/pcbs/leftsidereverse fix.kicad_pcb (KiCad board)
At the start: 2 copper layers, 153.4 x 89.2 mm, 70 parts

Commit message: pcbs finished for now
Parts:
- moved MCU1 9.50 mm to (233.0, 106.1)
- moved JST1 8.55 mm to (231.1, 128.5)
- moved RST1 6.85 mm to (250.1, 143.7)
- moved PWR1 6.01 mm to (250.1, 130.4)
- turned S23 to 180 degrees
- turned S24 to 180 degrees
- turned S25 to 180 degrees
- turned S26 to 180 degrees
- turned S27 to 180 degrees
- turned S28 to 180 degrees
- turned S29 to 180 degrees
- turned S30 to 180 degrees
- turned S31 to 180 degrees
- turned S32 to 180 degrees
- turned S33 to 180 degrees
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Connections:
- JST1 pad 1: BAT_P -> GND
- JST1 pad 2: GND -> BAT_P
- PWR1 pad 3: BAT_P -> (no net)
Routing:
- net JST1_2: track 3.60 -> 0.00 mm
- net JST1_1: track 3.60 -> 0.00 mm
